File: Kicad/DiscreteAmp.sch (KiCad schematic (older format))
At the start: 40 parts, among them J1 Conn_01x02_Female, J2 Conn_01x01_Female, J3 Conn_01x01_Female, J4 Conn_01x02_Female, Q1 2N3906, Q10 BD139, Q11 BD140, Q2 2N2219, Q3 2N2219, Q4 2N3906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

Commit message: fix
Parts:
- D1: footprint LED_THT:LED_D3.0mm -> LED_THT:LED_D5.0mm
- R4: value 2k2 -> 1k
Connections:
- net at Q11.1 (E), R17.1, R2.1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: now also J3.1 (Pin_1)
- net at R5.2: now also Q1.3 (C); no longer Q1.1 (E)
- net at R4.1: now also Q1.1 (E); no longer Q1.3 (C)
Other:
- moved on the sheet: J3
Changed lines of the file:
@@
 F 0 "D1" V 1839 3583 50  0000 R CNN
 F 1 "LED" V 1748 3583 50  0000 R CNN
-F 2 "LED_THT:LED_D3.0mm" H 1800 3700 50  0001 C CNN
+F 2 "LED_THT:LED_D5.0mm" H 1800 3700 50  0001 C CNN
 F 3 "~" H 1800 3700 50  0001 C CNN
 	1    1800 3700
@@
 F 3 "https://www.fairchildsemi.com/datasheets/2N/2N3906.pdf" H 2200 4150 50  0001 L CNN
 	1    2200 4150
-	1    0    0    -1
+	1    0    0    1
 $EndComp
 $Comp
@@
 P 2300 3700
 F 0 "R4" H 2230 3654 50  0000 R CNN
-F 1 "2k2" H 2230 3745 50  0000 R CNN
+F 1 "1k" H 2230 3745 50  0000 R CNN
 F 2 "Resistor_THT:R_Axial_DIN0207_L6.3mm_D2.5mm_P7.62mm_Horizontal" V 2230 3700 50  0001 C CNN
 F 3 "~" H 2300 3700 50  0001 C CNN
@@
 Connection ~ 3000 5200
 Wire Wire Line
-	3000 5200 5100 5200
+	3000 5200 3800 5200
 Wire Wire Line
 	2300 5150 2300 5200
@@
 L Connector:Conn_01x01_Female J3
 U 1 1 5EBA5C92
-P 3800 5400
-F 0 "J3" V 3738 5312 50  0000 R CNN
-F 1 "Conn_01x01_Female" V 3647 5312 50  0000 R CNN
-F 2 "Connector_Wire:SolderWirePad_1x01_Drill2.5mm" H 3800 5400 50  0001 C CNN
-F 3 "~" H 3800 5400 50  0001 C CNN
-	1    3800 5400
+P 3800 5450
+F 0 "J3" V 3738 5362 50  0000 R CNN
+F 1 "Conn_01x01_Female" V 3647 5362 50  0000 R CNN
+F 2 "Connector_Wire:SolderWirePad_1x01_Drill2.5mm" H 3800 5450 50  0001 C CNN
+F 3 "~" H 3800 5450 50  0001 C CNN
+	1    3800 5450
 	0    1    1    0
 $EndComp
+Wire Wire Line
+	3800 5250 3800 5200
+Connection ~ 3800 5200
+Wire Wire Line
+	3800 5200 5100 5200
 $EndSCHEMATC

Commit message: Fixed some 'bugs'
Parts:
- R10, R8: value 22R -> 100R
- R15: value 22R -> 180R
Connections:
- net at J3.1 (Pin_1), R17.1, R2.1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: now also Q11.2 (C); no longer Q11.1 (E)
- net at R19.1: now also Q11.1 (E); no longer Q11.2 (C)
Changed lines of the file:
@@
 P 3050 1350
 F 0 "R8" H 2980 1304 50  0000 R CNN
-F 1 "22R" H 2980 1395 50  0000 R CNN
+F 1 "100R" H 2980 1395 50  0000 R CNN
 F 2 "Resistor_THT:R_Axial_DIN0207_L6.3mm_D2.5mm_P7.62mm_Horizontal" V 2980 1350 50  0001 C CNN
 F 3 "~" H 3050 1350 50  0001 C CNN
@@
 P 3850 1350
 F 0 "R10" H 3780 1304 50  0000 R CNN
-F 1 "22R" H 3780 1395 50  0000 R CNN
+F 1 "100R" H 3780 1395 50  0000 R CNN
 F 2 "Resistor_THT:R_Axial_DIN0207_L6.3mm_D2.5mm_P7.62mm_Horizontal" V 3780 1350 50  0001 C CNN
 F 3 "~" H 3850 1350 50  0001 C CNN
@@
 P 5100 1350
 F 0 "R15" H 5030 1304 50  0000 R CNN
-F 1 "22R" H 5030 1395 50  0000 R CNN
+F 1 "180R" H 5030 1395 50  0000 R CNN
 F 2 "Resistor_THT:R_Axial_DIN0207_L6.3mm_D2.5mm_P7.62mm_Horizontal" V 5030 1350 50  0001 C CNN
 F 3 "~" H 5100 1350 50  0001 C CNN
@@
 F 3 "http://www.st.com/internet/com/TECHNICAL_RESOURCES/TECHNICAL_LITERATURE/DATASHEET/CD00001225.pdf" H 6000 3950 50  0001 L CNN
 	1    6000 3950
-	1    0    0    -1
+	1    0    0    1
 $EndComp
 $Comp
